File: Schematics/PCBS/ROMS.sch (EAGLE design)
At the start: 0 parts

Commit message: added 16mhz +grounding
Parts:
- added C1, C2: 20pF, SparkFun-Capacitors:20PF-0402T-50V-5%
- added IC1: ATMEGA328P-AU, ATMEGA328P-AU:ATMEGA328P-AU
- added Y1: 16MHz, SparkFun-Clocks:CRYSTAL-16MHZPTH-HC49US
Connections:
- new net GND: C1.1, C2.2
- new net N$1: C1.2, IC1.PB6_[PCINT6], Y1.2
- new net N$2: C2.1, IC1.PB7_[PCINT7], Y1.1
