File: Schematics/PCBS/ROMS.sch (EAGLE design)
At the start: 12 parts, among them IC1 ATMEGA328P-AU, M1 WIRELESS-NRF24L01-PA-EXT, Y1 16MHz

Commit message: Full Trigger test part started with just base PIR code
Connections:
- net IR_OUT: now also IC1.PC3_[PCINT11]
Changed lines of the file:
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@@
 <label x="-7.62" y="109.22" size="0.762" layer="95" xref="yes"/>
+</segment>
+<segment>
+<pinref part="IC1" gate="G$1" pin="PC3_[PCINT11]"/>
+<wire x1="81.28" y1="83.82" x2="81.28" y2="86.36" width="0.1524" layer="91"/>
+<label x="81.28" y="86.36" size="0.762" layer="95" rot="R90" xref="yes"/>
 </segment>
 </net>
