File: Schematics/PCBS/LC_Board.sch (EAGLE design)
At the start: 24 parts, among them IC1 ATMEGA328P-AU, Q10 220mA/50V/3.5Ω, U1 LT1763CS8-3.3#TRPBF

Commit message: LC_board PCB pos nearing finish for R1
Parts:
- removed JP2: switching from 5v RDI to 3.3v RDI input, pinhead:PINHD-1X3
- added SWITCHINGFROM5VRDITO3.3VRDIINPUT: (no value), adafruit:PINHD-1X3
Connections:
- net RDI: now also SWITCHINGFROM5VRDITO3.3VRDIINPUT.2; no longer JP2.2
- net RDI_3.3V: now also SWITCHINGFROM5VRDITO3.3VRDIINPUT.3; no longer JP2.3
- net RXD_IN: now also SWITCHINGFROM5VRDITO3.3VRDIINPUT.1; no longer JP2.1
Changed lines of the file:
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@@
 <part name="JP1" library="pinhead" library_urn="urn:adsk.eagle:library:325" deviceset="PINHD-1X8" device="" package3d_urn="urn:adsk.eagle:package:22409/2" value="IO"/>
 <part name="C2" library="SparkFun-Capacitors" library_urn="urn:adsk.eagle:library:510" deviceset="0.1UF" device="-0603-25V-(+80/-20%)" package3d_urn="urn:adsk.eagle:package:37414/1" value="0.1uF"/>
-<part name="JP2" library="pinhead" library_urn="urn:adsk.eagle:library:325" deviceset="PINHD-1X3" device="" package3d_urn="urn:adsk.eagle:package:22458/2" value="switching from 5v RDI to 3.3v RDI input"/>
 <part name="JP3" library="pinhead" library_urn="urn:adsk.eagle:library:325" deviceset="PINHD-1X3" device="" package3d_urn="urn:adsk.eagle:package:22458/2"/>
 <part name="CONVERTEPULLUP" library="audio amplifier example" library_urn="urn:adsk.eagle:library:970892" deviceset="R-US_" device="R0603" package3d_urn="urn:adsk.eagle:package:970938/2" value="10K"/>
 <part name="FRAME1" library="frames" library_urn="urn:adsk.eagle:library:229" deviceset="A3L-LOC" device=""/>
 <part name="RESET_PULLUP" library="audio amplifier example" library_urn="urn:adsk.eagle:library:970892" deviceset="R-US_" device="R0603" package3d_urn="urn:adsk.eagle:package:970938/2" value="10K"/>
+<part name="SWITCHINGFROM5VRDITO3.3VRDIINPUT" library="adafruit" library_urn="urn:adsk.eagle:library:420" deviceset="PINHD-1X3" device="" package3d_urn="urn:adsk.eagle:package:6240710/1"/>
 </parts>
 <sheets>
@@
 <attribute name="VALUE" x="563.499" y="34.544" size="1.778" layer="96" font="vector" rot="R90"/>
 </instance>
-<instance part="JP2" gate="A" x="436.88" y="-2.54" smashed="yes" rot="R270">
-<attribute name="VALUE" x="448.31" y="-5.08" size="0.8128" layer="96" rot="R180"/>
-</instance>
 <instance part="JP3" gate="A" x="474.98" y="-2.54" smashed="yes" rot="R270">
 <attribute name="VALUE" x="467.36" y="3.81" size="1.778" layer="96" rot="R270"/>
@@
 <attribute name="NAME" x="567.4614" y="39.37" size="1.778" layer="95" rot="R90"/>
 <attribute name="VALUE" x="572.262" y="39.37" size="1.778" layer="96" rot="R90"/>
+</instance>
+<instance part="SWITCHINGFROM5VRDITO3.3VRDIINPUT" gate="A" x="436.88" y="-2.54" smashed="yes" rot="R270">
+<attribute name="NAME" x="442.595" y="3.81" size="1.778" layer="95" rot="R270"/>
+<attribute name="VALUE" x="429.26" y="3.81" size="1.778" layer="96" rot="R270"/>
 </instance>
 </instances>
@@
 <pinref part="Q10" gate="NMOS" pin="D"/>
 <wire x1="439.42" y1="5.08" x2="439.42" y2="0" width="0.1524" layer="91"/>
-<pinref part="JP2" gate="A" pin="1"/>
+<pinref part="SWITCHINGFROM5VRDITO3.3VRDIINPUT" gate="A" pin="1"/>
 </segment>
 </net>
@@
 </segment>
 <segment>
-<pinref part="JP2" gate="A" pin="2"/>
 <wire x1="436.88" y1="5.08" x2="436.88" y2="0" width="0.1524" layer="91"/>
 <wire x1="431.8" y1="5.08" x2="436.88" y2="5.08" width="0.1524" layer="91"/>
 <label x="431.8" y="5.08" size="0.5588" layer="95" rot="R180" xref="yes"/>
+<pinref part="SWITCHINGFROM5VRDITO3.3VRDIINPUT" gate="A" pin="2"/>
 </segment>
 </net>
@@
 <net name="RDI_3.3V" class="0">
 <segment>
-<pinref part="JP2" gate="A" pin="3"/>
 <wire x1="434.34" y1="7.62" x2="434.34" y2="0" width="0.1524" layer="91"/>
 <wire x1="434.34" y1="7.62" x2="477.52" y2="7.62" width="0.1524" layer="91"/>
@@
 <wire x1="477.52" y1="7.62" x2="477.52" y2="0" width="0.1524" layer="91"/>
 <label x="434.34" y="7.62" size="0.8128" layer="95"/>
-</segment>
-</net>
+<pinref part="SWITCHINGFROM5VRDITO3.3VRDIINPUT" gate="A" pin="3"/>
+</segment>
+</net>

Commit message: Syncing schematic with board fixed
Parts:
- SWITCHINGFROM5VRDITO3.3VRDIINPUT: value (none) -> Switch4RXI INPUT; device adafruit:PINHD-1X3 -> pinhead:PINHD-1X3
Connections:
- net RDI renamed RXI
- net RDI_3.3V renamed RXI_3.3V
- removed net RDI2: IC1.PD0_[PCINT16], JP3.2
- new net PULLED_UP3.3VRX: CONVERTEPULLUP.2, JP3.3, Q10.S
- net D10: now also LED3BLUE.G; no longer LED2BLUE.G
- net D11: now also LED2GREEN.G; no longer LED3RED.G
- net D12: now also LED2RED.G; no longer LED3GREEN.G
- net D13: now also LED2BLUE.G; no longer LED3BLUE.G
- net D8: now also LED3RED.G; no longer LED2RED.G
- net D9: now also LED3GREEN.G; no longer LED2GREEN.G
- net RXI2: now also IC1.PD0_[PCINT16], JP3.2; no longer CONVERTEPULLUP.2, JP3.3, Q10.S
Changed lines of the file:
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@@
 <part name="FRAME1" library="frames" library_urn="urn:adsk.eagle:library:229" deviceset="A3L-LOC" device=""/>
 <part name="RESET_PULLUP" library="audio amplifier example" library_urn="urn:adsk.eagle:library:970892" deviceset="R-US_" device="R0603" package3d_urn="urn:adsk.eagle:package:970938/2" value="10K"/>
-<part name="SWITCHINGFROM5VRDITO3.3VRDIINPUT" library="adafruit" library_urn="urn:adsk.eagle:library:420" deviceset="PINHD-1X3" device="" package3d_urn="urn:adsk.eagle:package:6240710/1"/>
+<part name="SWITCHINGFROM5VRDITO3.3VRDIINPUT" library="pinhead" library_urn="urn:adsk.eagle:library:325" deviceset="PINHD-1X3" device="" package3d_urn="urn:adsk.eagle:package:22458/2" value="Switch4RXI INPUT"/>
 </parts>
 <sheets>
@@
 </instance>
 <instance part="SWITCHINGFROM5VRDITO3.3VRDIINPUT" gate="A" x="436.88" y="-2.54" smashed="yes" rot="R270">
-<attribute name="NAME" x="442.595" y="3.81" size="1.778" layer="95" rot="R270"/>
 <attribute name="VALUE" x="429.26" y="3.81" size="1.778" layer="96" rot="R270"/>
 </instance>
@@
 </segment>
 <segment>
+<pinref part="LED3GREEN" gate="G$1" pin="G"/>
+<wire x1="642.62" y1="-154.94" x2="642.62" y2="-165.1" width="0.1524" layer="91"/>
+<label x="642.62" y="-165.1" size="1.6764" layer="95" rot="R270" xref="yes"/>
+</segment>
+</net>
+<net name="D10" class="0">
+<segment>
+<pinref part="IC1" gate="G$1" pin="PB2_[PCINT2]"/>
+<wire x1="574.04" y1="-71.12" x2="574.04" y2="-73.66" width="0.1524" layer="91"/>
+<label x="574.04" y="-73.66" size="0.6096" layer="95" rot="R270" xref="yes"/>
+</segment>
+<segment>
+<pinref part="LED3BLUE" gate="G$1" pin="G"/>
+<wire x1="652.78" y1="-154.94" x2="652.78" y2="-165.1" width="0.1524" layer="91"/>
+<label x="652.78" y="-165.1" size="1.6764" layer="95" rot="R270" xref="yes"/>
+</segment>
+</net>
+<net name="D11" class="0">
+<segment>
+<pinref part="IC1" gate="G$1" pin="PB3_[PCINT3]"/>
+<wire x1="576.58" y1="-71.12" x2="576.58" y2="-73.66" width="0.1524" layer="91"/>
+<label x="576.58" y="-73.66" size="0.6096" layer="95" rot="R270" xref="yes"/>
+</segment>
+<segment>
 <pinref part="LED2GREEN" gate="G$1" pin="G"/>
 <wire x1="599.44" y1="-154.94" x2="599.44" y2="-165.1" width="0.1524" layer="91"/>
@@
 </segment>
 </net>
-<net name="D10" class="0">
-<segment>
-<pinref part="IC1" gate="G$1" pin="PB2_[PCINT2]"/>
-<wire x1="574.04" y1="-71.12" x2="574.04" y2="-73.66" width="0.1524" layer="91"/>
-<label x="574.04" y="-73.66" size="0.6096" layer="95" rot="R270" xref="yes"/>
+<net name="D12" class="0">
+<segment>
+<pinref part="IC1" gate="G$1" pin="PB4_[PCINT4]"/>
+<wire x1="579.12" y1="-71.12" x2="579.12" y2="-73.66" width="0.1524" layer="91"/>
+<label x="579.12" y="-73.66" size="0.6096" layer="95" rot="R270" xref="yes"/>
+</segment>
+<segment>
+<pinref part="LED2RED" gate="G$1" pin="G"/>
+<wire x1="589.28" y1="-154.94" x2="589.28" y2="-165.1" width="0.1524" layer="91"/>
+<label x="589.28" y="-165.1" size="1.6764" layer="95" rot="R270" xref="yes"/>
+</segment>
+</net>
+<net name="D13" class="0">
+<segment>
+<pinref part="IC1" gate="G$1" pin="PB5_[PCINT5]"/>
+<wire x1="599.44" y1="-43.18" x2="596.9" y2="-43.18" width="0.1524" layer="91"/>
+<label x="599.44" y="-43.18" size="0.6096" layer="95" xref="yes"/>
 </segment>
 <segment>
@@
 </segment>
 </net>
-<net name="D11" class="0">
-<segment>
-<pinref part="IC1" gate="G$1" pin="PB3_[PCINT3]"/>
-<wire x1="576.58" y1="-71.12" x2="576.58" y2="-73.66" width="0.1524" layer="91"/>
-<label x="576.58" y="-73.66" size="0.6096" layer="95" rot="R270" xref="yes"/>
+<net name="D8" class="0">
+<segment>
+<pinref part="IC1" gate="G$1" pin="PB0_[PCINT0]"/>
+<wire x1="568.96" y1="-71.12" x2="568.96" y2="-73.66" width="0.1524" layer="91"/>
+<label x="568.96" y="-73.66" size="0.6096" layer="95" rot="R270" xref="yes"/>
 </segment>
 <segment>
@@
 <wire x1="632.46" y1="-154.94" x2="632.46" y2="-165.1" width="0.1524" layer="91"/>
 <label x="632.46" y="-165.1" size="1.6764" layer="95" rot="R270" xref="yes"/>
-</segment>
-</net>
-<net name="D12" class="0">
-<segment>
-<pinref part="IC1" gate="G$1" pin="PB4_[PCINT4]"/>
-<wire x1="579.12" y1="-71.12" x2="579.12" y2="-73.66" width="0.1524" layer="91"/>
-<label x="579.12" y="-73.66" size="0.6096" layer="95" rot="R270" xref="yes"/>
-</segment>
-<segment>
-<pinref part="LED3GREEN" gate="G$1" pin="G"/>
-<wire x1="642.62" y1="-154.94" x2="642.62" y2="-165.1" width="0.1524" layer="91"/>
-<label x="642.62" y="-165.1" size="1.6764" layer="95" rot="R270" xref="yes"/>
-</segment>
-</net>
-<net name="D13" class="0">
-<segment>
-<pinref part="IC1" gate="G$1" pin="PB5_[PCINT5]"/>
-<wire x1="599.44" y1="-43.18" x2="596.9" y2="-43.18" width="0.1524" layer="91"/>
-<label x="599.44" y="-43.18" size="0.6096" layer="95" xref="yes"/>
-</segment>
-<segment>
-<pinref part="LED3BLUE" gate="G$1" pin="G"/>
-<wire x1="652.78" y1="-154.94" x2="652.78" y2="-165.1" width="0.1524" layer="91"/>
-<label x="652.78" y="-165.1" size="1.6764" layer="95" rot="R270" xref="yes"/>
-</segment>
-</net>
-<net name="D8" class="0">
-<segment>
-<pinref part="IC1" gate="G$1" pin="PB0_[PCINT0]"/>
-<wire x1="568.96" y1="-71.12" x2="568.96" y2="-73.66" width="0.1524" layer="91"/>
-<label x="568.96" y="-73.66" size="0.6096" layer="95" rot="R270" xref="yes"/>
-</segment>
-<segment>
-<pinref part="LED2RED" gate="G$1" pin="G"/>
-<wire x1="589.28" y1="-154.94" x2="589.28" y2="-165.1" width="0.1524" layer="91"/>
-<label x="589.28" y="-165.1" size="1.6764" layer="95" rot="R270" xref="yes"/>
 </segment>
 </net>
@@
 </segment>
 </net>
-<net name="RDI" class="0">
-<segment>
-<wire x1="452.12" y1="35.56" x2="457.2" y2="35.56" width="0.1524" layer="91"/>
-<label x="457.2" y="35.56" size="0.6096" layer="95" xref="yes"/>
-<pinref part="JP1" gate="A" pin="6"/>
-</segment>
-<segment>
-<wire x1="436.88" y1="5.08" x2="436.88" y2="0" width="0.1524" layer="91"/>
-<wire x1="431.8" y1="5.08" x2="436.88" y2="5.08" width="0.1524" layer="91"/>
-<label x="431.8" y="5.08" size="0.5588" layer="95" rot="R180" xref="yes"/>
-<pinref part="SWITCHINGFROM5VRDITO3.3VRDIINPUT" gate="A" pin="2"/>
-</segment>
-</net>
-<net name="RXI2" class="0">
+<net name="PULLED_UP3.3VRX" class="0">
 <segment>
 <wire x1="457.2" y1="5.08" x2="464.82" y2="5.08" width="0.1524" layer="91"/>
@@
 <wire x1="472.44" y1="5.08" x2="472.44" y2="0" width="0.1524" layer="91"/>
 <pinref part="CONVERTEPULLUP" gate="G$1" pin="2"/>
-</segment>
-</net>
-<net name="RDI2" class="0">
-<segment>
-<pinref part="IC1" gate="G$1" pin="PD0_[PCINT16]"/>
-<wire x1="566.42" y1="10.16" x2="566.42" y2="12.7" width="0.1524" layer="91"/>
-<label x="566.42" y="12.7" size="0.6096" layer="95" rot="R90" xref="yes"/>
-</segment>
-<segment>
-<label x="480.06" y="5.08" size="0.5588" layer="95" xref="yes"/>
-<wire x1="480.06" y1="5.08" x2="474.98" y2="5.08" width="0.1524" layer="91"/>
-<pinref part="JP3" gate="A" pin="2"/>
-<wire x1="474.98" y1="5.08" x2="474.98" y2="0" width="0.1524" layer="91"/>
-</segment>
-</net>
-<net name="RDI_3.3V" class="0">
+<label x="457.2" y="5.08" size="1.778" layer="95"/>
+</segment>
+</net>
+<net name="RXI_3.3V" class="0">
 <segment>
 <wire x1="434.34" y1="7.62" x2="434.34" y2="0" width="0.1524" layer="91"/>
@@
 </segment>
 </net>
+<net name="RXI" class="0">
+<segment>
+<wire x1="452.12" y1="35.56" x2="457.2" y2="35.56" width="0.1524" layer="91"/>
+<label x="457.2" y="35.56" size="0.6096" layer="95" xref="yes"/>
+<pinref part="JP1" gate="A" pin="6"/>
+</segment>
+<segment>
+<wire x1="436.88" y1="5.08" x2="436.88" y2="0" width="0.1524" layer="91"/>
+<wire x1="431.8" y1="5.08" x2="436.88" y2="5.08" width="0.1524" layer="91"/>
+<label x="431.8" y="5.08" size="0.5588" layer="95" rot="R180" xref="yes"/>
+<pinref part="SWITCHINGFROM5VRDITO3.3VRDIINPUT" gate="A" pin="2"/>
+</segment>
+</net>
+<net name="RXI2" class="0">
+<segment>
+<label x="480.06" y="5.08" size="0.5588" layer="95" xref="yes"/>
+<wire x1="480.06" y1="5.08" x2="474.98" y2="5.08" width="0.1524" layer="91"/>
+<pinref part="JP3" gate="A" pin="2"/>
+<wire x1="474.98" y1="5.08" x2="474.98" y2="0" width="0.1524" layer="91"/>
+</segment>
+<segment>
+<pinref part="IC1" gate="G$1" pin="PD0_[PCINT16]"/>
+<wire x1="566.42" y1="10.16" x2="566.42" y2="12.7" width="0.1524" layer="91"/>
+<label x="566.42" y="12.7" size="0.6096" layer="95" rot="R90" xref="yes"/>
+</segment>
+</net>
